File: electronics/Environment monitor/Environment_check.kicad_pcb (KiCad board)
At the start: 2 copper layers, 100 x 100 mm, 11 parts, among them J1 Audio_3.5mm, U1 ADS1115_ADS1015, U2 BM__80, U3 TSL2591, U4 ILI9341_2.8_TFT, U5 VEML6075

Commit message: Reopened with Kicad 5.99
Other:
- net class Apogee removed
- net class Default removed
- net class I2C removed
- net class Power removed
