File: electronics/Motor controller/RABR_motor_controller.kicad_pcb (KiCad board)
At the start: 2 copper layers, 113 x 99.1 mm, 47 parts, among them J1 Power In, M1 Shaft_motor, M2 Shaft_motor, M3 Shaft_motor, Q1 IRF9540N, SW1 Rotary_Encoder_Switch, SW2 SW_Push, SW3 SW_Push, SW4 SW_Push, U1 74HC14

Commit message: Reopened with Kicad 5.99
Other:
- net class Default removed
- net class Motor removed
- net class POWER removed
- net class Signal removed
